Commit message: adds legs with good tf

File: xpider_ws/src/xpider_descriptions/models/shield_bottom.xacro (robot description, xacro)
@@ -5,5 +5,5 @@
     <link name="shield_bottom">
     <visual>
-      <origin xyz="0 0 ${height_base}" rpy="0 -${m_pi_2} 0"/>
+      <origin xyz="0 0 0" rpy="0 -${m_pi_2} 0"/>
       <geometry>
         <mesh filename="package://xpider_descriptions/meshes/shield_bottom.stl" scale="${ratio_stl} ${ratio_stl} ${ratio_stl}"/>
@@ -12,5 +12,5 @@
       </visual>
       <collision>
-        <origin xyz="0 0 ${height_base}" rpy="0 -${m_pi_2} 0"/>
+        <origin xyz="0 0 0" rpy="0 -${m_pi_2} 0"/>
         <geometry>
           <mesh filename="package://xpider_descriptions/meshes/shield_bottom.stl" scale="${ratio_stl} ${ratio_stl} ${ratio_stl}"/>

File: xpider_ws/src/xpider_descriptions/models/shield_top.xacro (robot description, xacro)
@@ -5,5 +5,5 @@
     <link name="shield_top">
     <visual>
-      <origin xyz="0 0 ${height_base}" rpy="${m_pi_2} 0 0.07"/>
+      <origin xyz="0 0 0" rpy="${m_pi_2} 0 0.07"/>
       <geometry>
         <mesh filename="package://xpider_descriptions/meshes/shield_top.stl" scale="${ratio_stl} ${ratio_stl} ${ratio_stl}"/>
@@ -12,5 +12,5 @@
       </visual>
       <collision>
-        <origin xyz="0 0 ${height_base}" rpy="${m_pi_2} 0 0.07"/>
+        <origin xyz="0 0 0" rpy="${m_pi_2} 0 0.07"/>
         <geometry>
           <mesh filename="package://xpider_descriptions/meshes/shield_top.stl" scale="${ratio_stl} ${ratio_stl} ${ratio_stl}"/>

File: xpider_ws/src/xpider_descriptions/models/step.xacro (robot description, xacro)
@@ -5,5 +5,5 @@
     <link name="step">
     <visual>
-      <origin xyz="0 0 0.25" rpy="${m_pi_2} 0 ${m_pi_2}"/>
+      <origin xyz="0 0 -${height_step/2}" rpy="${m_pi_2} 0 ${m_pi_3}"/>
       <geometry>
         <mesh filename="package://xpider_descriptions/meshes/step.stl" scale="${ratio_stl} ${ratio_stl} ${ratio_stl}"/>
@@ -12,5 +12,5 @@
       </visual>
       <collision>
-        <origin xyz="0 0 0.25" rpy="${m_pi_2} 0 ${m_pi_2}"/>
+        <origin xyz="0 0 -${height_step/2}" rpy="${m_pi_2} 0 ${m_pi_3}"/>
         <geometry>
           <mesh filename="package://xpider_descriptions/meshes/step.stl" scale="${ratio_stl} ${ratio_stl} ${ratio_stl}"/>

File: xpider_ws/src/xpider_descriptions/models/step_base.xacro (robot description, xacro)
@@ -5,5 +5,5 @@
     <link name="step_base">
     <visual>
-      <origin xyz="0 0 ${height_base}" rpy="${m_pi_2} 0 ${m_pi_3}"/>
+      <origin xyz="0 0 0" rpy="${m_pi_2} 0 ${m_pi_3}"/>
       <geometry>
         <mesh filename="package://xpider_descriptions/meshes/step_base.stl" scale="${ratio_stl} ${ratio_stl} ${ratio_stl}"/>
@@ -12,5 +12,5 @@
       </visual>
       <collision>
-        <origin xyz="0 0 ${height_base}" rpy="${m_pi_2} 0 ${m_pi_3}"/>
+        <origin xyz="0 0 0" rpy="${m_pi_2} 0 ${m_pi_3}"/>
         <geometry>
           <mesh filename="package://xpider_descriptions/meshes/step_base.stl" scale="${ratio_stl} ${ratio_stl} ${ratio_stl}"/>

File: xpider_ws/src/xpider_descriptions/models/xpider.xacro (robot description, xacro)
@@ -3,9 +3,11 @@
 <xacro:include filename="$(find xpider_resources)/urdf/common_materials.xacro"/>
 <xacro:include filename="$(find xpider_resources)/urdf/common_constants.xacro"/>
+<xacro:include filename="$(find xpider_descriptions)/models/step_bridge.xacro"/>
+<xacro:include filename="$(find xpider_descriptions)/models/leg.xacro"/>
   <xacro:include filename="$(find xpider_descriptions)/models/base_link.xacro"/>
   <joint name="base_joint" type="fixed">
 		<parent link="base_link" />
 		<child link="shield_top" />
-		<origin xyz="0 0 0" rpy="0 0 0" />
+		<origin xyz="0 0 ${height_base}" rpy="0 0 ${m_pi_3}" /> <!-- TOCHECK-->
 	</joint>
   <xacro:include filename="$(find xpider_descriptions)/models/shield_top.xacro"/>
@@ -13,5 +15,5 @@
 		<parent link="base_link" />
 		<child link="shield_bottom" />
-		<origin xyz="0 0 0" rpy="0 0 0" />
+		<origin xyz="0 0 ${height_base}" rpy="0 0 ${m_pi_3 + m_pi_6}" />
 	</joint>
   <xacro:include filename="$(find xpider_descriptions)/models/shield_bottom.xacro"/>
@@ -19,12 +21,31 @@
 		<parent link="base_link" />
 		<child link="step" />
-		<origin xyz="0 0 0" rpy="0 0 0" />
+		<origin xyz="0 0 ${base_link_to_step_height + height_step/2}" rpy="0 0 ${m_pi_2 + m_pi_6}" />
 	</joint>
-  <xacro:include filename="$(find xpider_descriptions)/models/step.xacro"/>
+   <xacro:include filename="$(find xpider_descriptions)/models/step.xacro"/>
   <joint name="base_joint4" type="fixed">
 		<parent link="base_link" />
 		<child link="step_base" />
-		<origin xyz="0 0 0" rpy="0 0 0" />
+		<origin xyz="0 0 ${height_base}" rpy="0 0 ${m_pi_3 + m_pi_6}" />
 	</joint>
   <xacro:include filename="$(find xpider_descriptions)/models/step_base.xacro"/>
+  <!--  Legs -->
+  <joint name="base_link_to_leg_1" type="fixed">
+		<parent link="base_link" />
+		<child link="leg_1" />
+    <origin xyz="${diameter_step} 0 ${base_link_to_step_height + height_step/2 + 0.013}" rpy="0 0 0"/>
+	</joint>
+  <xacro:leg num="1"/>
+  <joint name="base_link_to_leg_2" type="fixed">
+		<parent link="base_link" />
+		<child link="leg_2" />
+    <origin xyz="${diameter_step*cos_m_2_pi_3} ${diameter_step*sin_m_2_pi_3} ${base_link_to_step_height + height_step/2}" rpy="0 0 ${m_2_pi_3}"/>
+	</joint>
+  <xacro:leg num="2"/>
+  <joint name="base_link_to_leg_3" type="fixed">
+		<parent link="base_link" />
+		<child link="leg_3" />
+    <origin xyz="${diameter_step*cos_m_4_pi_3} ${diameter_step*sin_m_4_pi_3} ${base_link_to_step_height + height_step/2}" rpy="0 0 ${2*m_2_pi_3}"/>
+	</joint>
+  <xacro:leg num="3"/>
 </robot>

File: xpider_ws/src/xpider_resources/urdf/common_constants.xacro (robot description, xacro)
@@ -7,9 +7,20 @@
   <!-- 3Pi divided by two -->
   <xacro:property name="m_3_pi_2" value="2.35619449" />
+  <!-- 3Pi divided by two -->
+  <xacro:property name="m_2_pi_3" value="2.09439510239" />
   <!-- Pi divided by four -->
   <xacro:property name="m_pi_4" value="0.785398163" />
   <!-- Pi divided by three -->
   <xacro:property name="m_pi_3" value="1.0471975512" />
+  <!-- Pi divided by six -->
+  <xacro:property name="m_pi_6" value="0.52359877559" />
+  <xacro:property name="cos_m_2_pi_3" value="-0.5" />
+  <xacro:property name="sin_m_2_pi_3" value="0.86602540378" />
+  <xacro:property name="cos_m_4_pi_3" value="-0.5" />
+  <xacro:property name="sin_m_4_pi_3" value="-0.86602540378" />
   <xacro:property name="ratio_stl" value="0.01006046568"/>
   <xacro:property name="height_base" value="0.53"/>
+  <xacro:property name="height_step" value="0.04"/>
+  <xacro:property name="base_link_to_step_height" value="0.27"/>
+  <xacro:property name="diameter_step" value="0.5425" />
 </robot>
