Commit message: corrected leg stl, starts step_up

File: xpider_ws/src/xpider_descriptions/models/leg.xacro (robot description, xacro)
@@ -3,17 +3,19 @@
 <xacro:include filename="$(find xpider_resources)/urdf/common_materials.xacro"/>
 <xacro:include filename="$(find xpider_resources)/urdf/common_constants.xacro"/>
+<xacro:include filename="$(find xpider_resources)/urdf/common_colours.xacro"/>
     <xacro:macro name="leg" params="num">
       <link name="leg_${num}">
       <visual>
-        <origin xyz="-${diameter_step-0.015} 0 0.029" rpy="0 -${m_pi_2} 0"/>
+        <origin xyz="0 0 0" rpy="0 -${m_pi-m_pi_6*0.5} 0"/>
         <geometry>
           <mesh filename="package://xpider_descriptions/meshes/leg.stl" scale="${ratio_stl} ${ratio_stl} ${ratio_stl}"/>
+          <xacro:material_xpider_yellow />
         </geometry>
-        <xacro:material_xpider_grey />
         </visual>
         <collision>
-          <origin xyz="-${diameter_step-0.015} 0 0.029" rpy="0 -${m_pi_2} 0"/>
+          <origin xyz="0 0 0" rpy="0 -${m_pi-m_pi_6*0.5} 0"/>
           <geometry>
             <mesh filename="package://xpider_descriptions/meshes/leg.stl" scale="${ratio_stl} ${ratio_stl} ${ratio_stl}"/>
+            <xacro:material_xpider_yellow />
           </geometry>
         </collision>

File: xpider_ws/src/xpider_descriptions/models/xpider.xacro (robot description, xacro)
@@ -5,4 +5,6 @@
 <xacro:include filename="$(find xpider_descriptions)/models/step_bridge.xacro"/>
 <xacro:include filename="$(find xpider_descriptions)/models/leg.xacro"/>
+<xacro:include filename="$(find xpider_descriptions)/models/step_up.xacro"/>
+<!--<xacro:include filename="$(find xpider_descriptions)/models/leg_shield.xacro"/>-->
   <xacro:include filename="$(find xpider_descriptions)/models/base_link.xacro"/>
   <joint name="base_joint" type="fixed">
@@ -34,5 +36,5 @@
 		<parent link="base_link" />
 		<child link="leg_1" />
-    <origin xyz="${diameter_step} 0 ${base_link_to_step_height + height_step/2 + 0.013}" rpy="0 0 0"/>
+    <origin xyz="${diameter_step} 0 ${base_link_to_step_height + height_leg}" rpy="0 0 0"/>
 	</joint>
   <xacro:leg num="1"/>
@@ -49,3 +51,36 @@
 	</joint>
   <xacro:leg num="3"/>
+  <joint name="base_link_to_step_up_1" type="fixed">
+		<parent link="base_link" />
+		<child link="step_up_1" />
+    <origin xyz="${diameter_step_up} 0 ${base_link_to_up}" rpy="0 ${m_pi_6} 0"/>
+	</joint>
+  <xacro:step_up num="1"/>
+<!--  <joint name="base_link_to_leg_4" type="fixed">
+		<parent link="base_link" />
+		<child link="leg_4" />
+    <origin xyz="0 0 0" rpy="0 ${m_pi} 0"/>
+	</joint>
+        <link name="leg_4">
+      <visual>
+        <origin xyz="0 0 0" rpy="0 0 0"/>
+        <geometry>
+          <mesh filename="package://xpider_descriptions/meshes/leg.stl" scale="${ratio_stl} ${ratio_stl} ${ratio_stl}"/>
+          <xacro:color_xpider_white />
+        </geometry>
+        </visual>
+        <collision>
+          <origin xyz="0 0 0" rpy="0 0 0"/>
+          <geometry>
+            <mesh filename="package://xpider_descriptions/meshes/leg.stl" scale="${ratio_stl} ${ratio_stl} ${ratio_stl}"/>
+            <xacro:color_xpider_white />
+          </geometry>
+        </collision>
+      </link>-->
+<!--   <joint name="base_link_to_leg_shield_3" type="fixed">
+		<parent link="leg_1" />
+		<child link="leg_shield_1" />
+    <origin xyz="0 0 0" rpy="-${m_pi_2} 0 0"/>
+	</joint>
+  <xacro:leg_shield num="1"/>-->
 </robot>

File: xpider_ws/src/xpider_resources/urdf/common_constants.xacro (robot description, xacro)
@@ -22,5 +22,8 @@
   <xacro:property name="height_base" value="0.53"/>
   <xacro:property name="height_step" value="0.04"/>
-  <xacro:property name="base_link_to_step_height" value="0.27"/>
-  <xacro:property name="diameter_step" value="0.5425" />
+  <xacro:property name="height_leg" value="${height_step/2 + 0.007}"/>
+  <xacro:property name="base_link_to_step_height" value="0.25"/>
+  <xacro:property name="base_link_to_up" value="0.499"/>
+  <xacro:property name="diameter_step" value="0.541" />
+  <xacro:property name="diameter_step_up" value="${26*ratio_stl}" />
 </robot>
