Commit message: adds step_base

File: xpider_ws/src/xpider_descriptions/models/base_link.xacro (robot description, xacro)
@@ -5,5 +5,5 @@
     <link name="base_link">
     <visual>
-      <origin xyz="0 0 0.53" rpy="0 0 0"/>
+      <origin xyz="0 0 ${height_base}" rpy="0 0 0"/>
       <geometry>
         <mesh filename="package://xpider_descriptions/meshes/base_link.stl" scale="${ratio_stl} ${ratio_stl} ${ratio_stl}"/>
@@ -12,5 +12,5 @@
       </visual>
       <collision>
-        <origin xyz="0 0 0.53" rpy="0 0 0"/>
+        <origin xyz="0 0 ${height_base}" rpy="0 0 0"/>
         <geometry>
           <mesh filename="package://xpider_descriptions/meshes/base_link.stl" scale="${ratio_stl} ${ratio_stl} ${ratio_stl}"/>

File: xpider_ws/src/xpider_descriptions/models/shield_bottom.xacro (robot description, xacro)
@@ -5,5 +5,5 @@
     <link name="shield_bottom">
     <visual>
-      <origin xyz="0 0 0.53" rpy="0 -${m_pi_2} 0"/>
+      <origin xyz="0 0 ${height_base}" rpy="0 -${m_pi_2} 0"/>
       <geometry>
         <mesh filename="package://xpider_descriptions/meshes/shield_bottom.stl" scale="${ratio_stl} ${ratio_stl} ${ratio_stl}"/>
@@ -12,5 +12,5 @@
       </visual>
       <collision>
-        <origin xyz="0 0 0.53" rpy="0 -${m_pi_2} 0"/>
+        <origin xyz="0 0 ${height_base}" rpy="0 -${m_pi_2} 0"/>
         <geometry>
           <mesh filename="package://xpider_descriptions/meshes/shield_bottom.stl" scale="${ratio_stl} ${ratio_stl} ${ratio_stl}"/>

File: xpider_ws/src/xpider_descriptions/models/shield_top.xacro (robot description, xacro)
@@ -5,5 +5,5 @@
     <link name="shield_top">
     <visual>
-      <origin xyz="0 0 0.53" rpy="${m_pi_2} 0 0.07"/>
+      <origin xyz="0 0 ${height_base}" rpy="${m_pi_2} 0 0.07"/>
       <geometry>
         <mesh filename="package://xpider_descriptions/meshes/shield_top.stl" scale="${ratio_stl} ${ratio_stl} ${ratio_stl}"/>
@@ -12,5 +12,5 @@
       </visual>
       <collision>
-        <origin xyz="0 0 0.53" rpy="${m_pi_2} 0 0.07"/>
+        <origin xyz="0 0 ${height_base}" rpy="${m_pi_2} 0 0.07"/>
         <geometry>
           <mesh filename="package://xpider_descriptions/meshes/shield_top.stl" scale="${ratio_stl} ${ratio_stl} ${ratio_stl}"/>

File: xpider_ws/src/xpider_descriptions/models/xpider.xacro (robot description, xacro)
@@ -22,3 +22,9 @@
 	</joint>
   <xacro:include filename="$(find xpider_descriptions)/models/step.xacro"/>
+  <joint name="base_joint4" type="fixed">
+		<parent link="base_link" />
+		<child link="step_base" />
+		<origin xyz="0 0 0" rpy="0 0 0" />
+	</joint>
+  <xacro:include filename="$(find xpider_descriptions)/models/step_base.xacro"/>
 </robot>

File: xpider_ws/src/xpider_resources/urdf/common_constants.xacro (robot description, xacro)
@@ -9,4 +9,7 @@
   <!-- Pi divided by four -->
   <xacro:property name="m_pi_4" value="0.785398163" />
+  <!-- Pi divided by three -->
+  <xacro:property name="m_pi_3" value="1.0471975512" />
   <xacro:property name="ratio_stl" value="0.01006046568"/>
+  <xacro:property name="height_base" value="0.53"/>
 </robot>

Commit message: each link depends on each other

File: xpider_ws/src/xpider_descriptions/models/base_link.xacro (robot description, xacro)
@@ -9,5 +9,5 @@
         <mesh filename="package://xpider_descriptions/meshes/base_link.stl" scale="${ratio_stl} ${ratio_stl} ${ratio_stl}"/>
       </geometry>
-      <xacro:material_xpider_grey />
+      <xacro:material_xpider_greyish />
       </visual>
       <collision>

File: xpider_ws/src/xpider_descriptions/models/leg.xacro (robot description, xacro)
@@ -7,16 +7,16 @@
       <link name="leg_${num}">
       <visual>
-        <origin xyz="0 0 0" rpy="0 -${m_pi-m_pi_6*0.5} 0"/>
+        <origin xyz="0 0 0" rpy="0 -${m_pi-m_pi_6*0.3} 0"/>
         <geometry>
           <mesh filename="package://xpider_descriptions/meshes/leg.stl" scale="${ratio_stl} ${ratio_stl} ${ratio_stl}"/>
-          <xacro:material_xpider_yellow />
         </geometry>
+        <xacro:material_xpider_greyish />
         </visual>
         <collision>
-          <origin xyz="0 0 0" rpy="0 -${m_pi-m_pi_6*0.5} 0"/>
+          <origin xyz="0 0 0" rpy="0 -${m_pi-m_pi_6*0.3} 0"/>
           <geometry>
             <mesh filename="package://xpider_descriptions/meshes/leg.stl" scale="${ratio_stl} ${ratio_stl} ${ratio_stl}"/>
-            <xacro:material_xpider_yellow />
           </geometry>
+          <xacro:material_xpider_greyish/>
         </collision>
       </link>

File: xpider_ws/src/xpider_descriptions/models/leg_shield.xacro (robot description, xacro)
@@ -10,5 +10,5 @@
           <mesh filename="package://xpider_descriptions/meshes/leg_shield.stl" scale="${ratio_stl} ${ratio_stl} ${ratio_stl}"/>
         </geometry>
-        <xacro:color_xpider_white />
+        <xacro:material_xpider_greyish />
         </visual>
         <collision>

File: xpider_ws/src/xpider_descriptions/models/shield_bottom.xacro (robot description, xacro)
@@ -9,5 +9,5 @@
         <mesh filename="package://xpider_descriptions/meshes/shield_bottom.stl" scale="${ratio_stl} ${ratio_stl} ${ratio_stl}"/>
       </geometry>
-      <xacro:material_xpider_grey />
+      <xacro:material_xpider_greyish />
       </visual>
       <collision>

File: xpider_ws/src/xpider_descriptions/models/shield_top.xacro (robot description, xacro)
@@ -9,5 +9,5 @@
         <mesh filename="package://xpider_descriptions/meshes/shield_top.stl" scale="${ratio_stl} ${ratio_stl} ${ratio_stl}"/>
       </geometry>
-      <xacro:material_xpider_grey />
+      <xacro:material_xpider_greyish />
       </visual>
       <collision>

File: xpider_ws/src/xpider_descriptions/models/step_up.xacro (robot description, xacro)
@@ -6,5 +6,5 @@
     <link name="step_up_${num}">
     <visual>
-      <origin xyz="0 0 -${height_step/2}" rpy="${m_pi_2} 0 ${m_pi_3+m_pi_6}"/>
+      <origin xyz="0 0 0" rpy="${m_pi_2-0.2} 0 ${m_pi_3+m_pi_6}"/>
       <geometry>
         <mesh filename="package://xpider_descriptions/meshes/step_up.stl" scale="${ratio_stl} ${ratio_stl} ${ratio_stl}"/>
@@ -13,5 +13,5 @@
       </visual>
       <collision>
-        <origin xyz="0 0 -${height_step/2}" rpy="${m_pi_2} 0 ${m_pi_3+m_pi_6}"/>
+        <origin xyz="0 0 0" rpy="${m_pi_2-0.2} 0 ${m_pi_3+m_pi_6}"/>
         <geometry>
           <mesh filename="package://xpider_descriptions/meshes/step_up.stl" scale="${ratio_stl} ${ratio_stl} ${ratio_stl}"/>

File: xpider_ws/src/xpider_descriptions/models/xpider.xacro (robot description, xacro)
@@ -54,7 +54,19 @@
 		<parent link="base_link" />
 		<child link="step_up_1" />
-    <origin xyz="${diameter_step_up} 0 ${base_link_to_up}" rpy="0 ${m_pi_6} 0"/>
+    <origin xyz="${diameter_step_up} 0 ${base_link_to_step_up}" rpy="0 ${m_pi_6} 0"/>
 	</joint>
   <xacro:step_up num="1"/>
+  <joint name="base_link_to_step_up_2" type="fixed">
+		<parent link="base_link" />
+		<child link="step_up_2" />
+    <origin xyz="${diameter_step_up*cos_m_2_pi_3} ${diameter_step_up*sin_m_2_pi_3} ${base_link_to_step_up}" rpy="0 ${m_pi_6} ${m_2_pi_3}"/>
+	</joint>
+  <xacro:step_up num="2"/>
+  <joint name="base_link_to_step_up_3" type="fixed">
+		<parent link="base_link" />
+		<child link="step_up_3" />
+    <origin xyz="${diameter_step_up*cos_m_4_pi_3} ${diameter_step_up*sin_m_4_pi_3} ${base_link_to_step_up}" rpy="0 ${m_pi_6} ${2*m_2_pi_3}"/>
+	</joint>
+  <xacro:step_up num="3"/>
 <!--  <joint name="base_link_to_leg_4" type="fixed">
 		<parent link="base_link" />

File: xpider_ws/src/xpider_resources/urdf/common_constants.xacro (robot description, xacro)
@@ -20,10 +20,10 @@
   <xacro:property name="sin_m_4_pi_3" value="-0.86602540378" />
   <xacro:property name="ratio_stl" value="0.01006046568"/>
-  <xacro:property name="height_base" value="0.53"/>
+  <xacro:property name="height_base" value="${48.705498889*ratio_stl}"/>
   <xacro:property name="height_step" value="0.04"/>
   <xacro:property name="height_leg" value="${height_step/2 + 0.007}"/>
-  <xacro:property name="base_link_to_step_height" value="0.25"/>
-  <xacro:property name="base_link_to_up" value="0.499"/>
-  <xacro:property name="diameter_step" value="0.541" />
+  <xacro:property name="base_link_to_step_height" value="${height_base-0.28}"/>
+  <xacro:property name="base_link_to_step_up" value="${height_base - 0.05}"/>
+  <xacro:property name="diameter_step" value="${53.7748467325*ratio_stl}" />
   <xacro:property name="diameter_step_up" value="${26*ratio_stl}" />
 </robot>

Commit message: adds gazebo support

File: xpider_ws/src/xpider_descriptions/models/base_link.xacro (robot description, xacro)
@@ -17,4 +17,12 @@
         </geometry>
       </collision>
+      <inertial>
+      <origin xyz="0 0 ${height_base}" rpy="0 0 0"/>
+      <mass value="1"/>
+      <inertia
+        ixx="1.0" ixy="0.0" ixz="0.0"
+        iyy="1.0" iyz="0.0"
+        izz="1.0"/>
+    </inertial>
     </link>
 </robot>

File: xpider_ws/src/xpider_descriptions/models/shield_bottom.xacro (robot description, xacro)
@@ -1,4 +1,4 @@
 <?xml version="1.0" ?>
-<robot name="xpider_base_link" xmlns:xacro="http://ros.org/wiki/xacro">
+<robot name="xpider_shield_bottom" xmlns:xacro="http://ros.org/wiki/xacro">
 <xacro:include filename="$(find xpider_resources)/urdf/common_materials.xacro"/>
 <xacro:include filename="$(find xpider_resources)/urdf/common_constants.xacro"/>

File: xpider_ws/src/xpider_descriptions/models/shield_top.xacro (robot description, xacro)
@@ -1,4 +1,4 @@
 <?xml version="1.0" ?>
-<robot name="xpider_base_link" xmlns:xacro="http://ros.org/wiki/xacro">
+<robot name="xpider_shield_top" xmlns:xacro="http://ros.org/wiki/xacro">
 <xacro:include filename="$(find xpider_resources)/urdf/common_materials.xacro"/>
 <xacro:include filename="$(find xpider_resources)/urdf/common_constants.xacro"/>

File: xpider_ws/src/xpider_descriptions/models/xpider.xacro (robot description, xacro)
@@ -1,4 +1,4 @@
 <?xml version="1.0" ?>
-<robot name="xpider_shield_top_base_link" xmlns:xacro="http://ros.org/wiki/xacro">
+<robot name="xpider" xmlns:xacro="http://ros.org/wiki/xacro">
 <xacro:include filename="$(find xpider_resources)/urdf/common_materials.xacro"/>
 <xacro:include filename="$(find xpider_resources)/urdf/common_constants.xacro"/>
@@ -6,5 +6,11 @@
 <xacro:include filename="$(find xpider_descriptions)/models/leg.xacro"/>
 <xacro:include filename="$(find xpider_descriptions)/models/step_up.xacro"/>
+<xacro:include filename="$(find xpider_descriptions)/models/xpider.gazebo" />
 <!--<xacro:include filename="$(find xpider_descriptions)/models/leg_shield.xacro"/>-->
+  <link name="world"/>
+  <joint name="fixed" type="fixed">
+    <parent link="world"/>
+    <child link="base_link"/>
+  </joint>
   <xacro:include filename="$(find xpider_descriptions)/models/base_link.xacro"/>
   <joint name="base_joint" type="fixed">
