Commit message: adds step, clean xacros/launch

File: xpider_ws/src/xpider_descriptions/models/xpider.xacro (robot description, xacro)
@@ -10,3 +10,15 @@
 	</joint>
   <xacro:include filename="$(find xpider_descriptions)/models/shield_top.xacro"/>
+  <joint name="base_joint2" type="fixed">
+		<parent link="base_link" />
+		<child link="shield_bottom" />
+		<origin xyz="0 0 0" rpy="0 0 0" />
+	</joint>
+  <xacro:include filename="$(find xpider_descriptions)/models/shield_bottom.xacro"/>
+  <joint name="base_joint3" type="fixed">
+		<parent link="base_link" />
+		<child link="step" />
+		<origin xyz="0 0 0" rpy="0 0 0" />
+	</joint>
+  <xacro:include filename="$(find xpider_descriptions)/models/step.xacro"/>
 </robot>

File: xpider_ws/src/xpider_resources/urdf/common_constants.xacro (robot description, xacro)
@@ -5,4 +5,6 @@
   <!-- Pi divided by two -->
   <xacro:property name="m_pi_2" value="1.570796327" />
+  <!-- 3Pi divided by two -->
+  <xacro:property name="m_3_pi_2" value="2.35619449" />
   <!-- Pi divided by four -->
   <xacro:property name="m_pi_4" value="0.785398163" />

Commit message: adds step_connect 1 2 3

File: xpider_ws/src/xpider_descriptions/models/xpider.xacro (robot description, xacro)
@@ -6,4 +6,5 @@
 <xacro:include filename="$(find xpider_descriptions)/models/leg.xacro"/>
 <xacro:include filename="$(find xpider_descriptions)/models/step_up.xacro"/>
+<xacro:include filename="$(find xpider_descriptions)/models/step_connect.xacro"/>
 <xacro:include filename="$(find xpider_descriptions)/models/xpider.gazebo" />
 <!--<xacro:include filename="$(find xpider_descriptions)/models/leg_shield.xacro"/>-->
@@ -38,5 +39,5 @@
 	</joint>
   <xacro:include filename="$(find xpider_descriptions)/models/step_base.xacro"/>
-  <!--  Legs -->
+  <!--  First set of Legs -->
   <joint name="base_link_to_leg_1" type="fixed">
 		<parent link="base_link" />
@@ -75,30 +76,22 @@
 	</joint>
   <xacro:step_up num="3"/>
-<!--  <joint name="base_link_to_leg_4" type="fixed">
+ <!-- Second set of legs -->
+  <joint name="base_link_to_step_connect_1" type="fixed">
 		<parent link="base_link" />
-		<child link="leg_4" />
-    <origin xyz="0 0 0" rpy="0 ${m_pi} 0"/>
+		<child link="step_connect_1" />
+    <origin xyz="${diameter_step_connect*cos_m_pi_3} ${diameter_step_connect*sin_m_pi_3} ${base_link_to_step_height + 0.0624}" rpy="0 0 ${-m_pi_6}"/>
 	</joint>
-        <link name="leg_4">
-      <visual>
-        <origin xyz="0 0 0" rpy="0 0 0"/>
-        <geometry>
-          <mesh filename="package://xpider_descriptions/meshes/leg.stl" scale="${ratio_stl} ${ratio_stl} ${ratio_stl}"/>
-          <xacro:color_xpider_white />
-        </geometry>
-        </visual>
-        <collision>
-          <origin xyz="0 0 0" rpy="0 0 0"/>
-          <geometry>
-            <mesh filename="package://xpider_descriptions/meshes/leg.stl" scale="${ratio_stl} ${ratio_stl} ${ratio_stl}"/>
-            <xacro:color_xpider_white />
-          </geometry>
-        </collision>
-      </link>-->
-<!--   <joint name="base_link_to_leg_shield_3" type="fixed">
-		<parent link="leg_1" />
-		<child link="leg_shield_1" />
-    <origin xyz="0 0 0" rpy="-${m_pi_2} 0 0"/>
+  <xacro:step_connect num="1"/>
+    <joint name="base_link_to_step_connect_2" type="fixed">
+		<parent link="base_link" />
+		<child link="step_connect_2" />
+    <origin xyz="${diameter_step_connect*cos_m_pi} ${diameter_step_connect*sin_m_pi} ${base_link_to_step_height + 0.0624}" rpy="0 0 ${-m_pi_6 + m_2_pi_3}"/>
 	</joint>
-  <xacro:leg_shield num="1"/>-->
+  <xacro:step_connect num="2"/>
+    <joint name="base_link_to_step_connect_3" type="fixed">
+		<parent link="base_link" />
+		<child link="step_connect_3" />
+    <origin xyz="${diameter_step_connect*cos_m_5_pi_3} ${diameter_step_connect*sin_m_5_pi_3} ${base_link_to_step_height + 0.0624}" rpy="0 0 ${-m_pi_6 + 2*m_2_pi_3}"/>
+	</joint>
+  <xacro:step_connect num="3"/>
 </robot>

File: xpider_ws/src/xpider_resources/urdf/common_constants.xacro (robot description, xacro)
@@ -15,8 +15,14 @@
   <!-- Pi divided by six -->
   <xacro:property name="m_pi_6" value="0.52359877559" />
+  <xacro:property name="cos_m_pi" value="-1" />
+  <xacro:property name="sin_m_pi" value="0" />
+  <xacro:property name="cos_m_pi_3" value="0.5" />
+  <xacro:property name="sin_m_pi_3" value="0.86602540378" />
   <xacro:property name="cos_m_2_pi_3" value="-0.5" />
   <xacro:property name="sin_m_2_pi_3" value="0.86602540378" />
   <xacro:property name="cos_m_4_pi_3" value="-0.5" />
   <xacro:property name="sin_m_4_pi_3" value="-0.86602540378" />
+  <xacro:property name="cos_m_5_pi_3" value="0.5" />
+  <xacro:property name="sin_m_5_pi_3" value="-0.86602540378" />
   <xacro:property name="ratio_stl" value="0.01006046568"/>
   <xacro:property name="height_base" value="${48.705498889*ratio_stl}"/>
@@ -27,3 +33,4 @@
   <xacro:property name="diameter_step" value="${53.7748467325*ratio_stl}" />
   <xacro:property name="diameter_step_up" value="${26*ratio_stl}" />
+  <xacro:property name="diameter_step_connect" value="${5.5*ratio_stl}" />
 </robot>

Commit message: adds step_b 1 2 3

File: xpider_ws/src/xpider_descriptions/models/xpider.xacro (robot description, xacro)
@@ -7,4 +7,5 @@
 <xacro:include filename="$(find xpider_descriptions)/models/step_up.xacro"/>
 <xacro:include filename="$(find xpider_descriptions)/models/step_connect.xacro"/>
+<xacro:include filename="$(find xpider_descriptions)/models/step_b.xacro"/>
 <xacro:include filename="$(find xpider_descriptions)/models/xpider.gazebo" />
 <!--<xacro:include filename="$(find xpider_descriptions)/models/leg_shield.xacro"/>-->
@@ -83,5 +84,5 @@
 	</joint>
   <xacro:step_connect num="1"/>
-    <joint name="base_link_to_step_connect_2" type="fixed">
+  <joint name="base_link_to_step_connect_2" type="fixed">
 		<parent link="base_link" />
 		<child link="step_connect_2" />
@@ -89,5 +90,5 @@
 	</joint>
   <xacro:step_connect num="2"/>
-    <joint name="base_link_to_step_connect_3" type="fixed">
+  <joint name="base_link_to_step_connect_3" type="fixed">
 		<parent link="base_link" />
 		<child link="step_connect_3" />
@@ -95,3 +96,21 @@
 	</joint>
   <xacro:step_connect num="3"/>
+  <joint name="step_connect_1_to_step_b_1" type="fixed">
+		<parent link="step_connect_1" />
+		<child link="step_b_1" />
+    <origin xyz="${0} ${0.042} ${0.0402}" rpy="0 0 ${0}"/>
+	</joint>
+  <xacro:step_b num="1"/>
+    <joint name="step_connect_2_to_step_b_2" type="fixed">
+		<parent link="step_connect_2" />
+		<child link="step_b_2" />
+    <origin xyz="${0} ${diameter_step_connect_to_step_b} ${height_step_connect_to_step_b}" rpy="0 0 0"/>
+	</joint>
+  <xacro:step_b num="2"/>
+    <joint name="step_connect_3_to_step_b_3" type="fixed">
+		<parent link="step_connect_3" />
+		<child link="step_b_3" />
+    <origin xyz="${0} ${diameter_step_connect_to_step_b} ${height_step_connect_to_step_b}" rpy="0 0 0"/>
+	</joint>
+  <xacro:step_b num="3"/>
 </robot>

File: xpider_ws/src/xpider_resources/urdf/common_constants.xacro (robot description, xacro)
@@ -34,3 +34,5 @@
   <xacro:property name="diameter_step_up" value="${26*ratio_stl}" />
   <xacro:property name="diameter_step_connect" value="${5.5*ratio_stl}" />
+  <xacro:property name="height_step_connect_to_step_b" value="${3.99583888844*ratio_stl}" />
+  <xacro:property name="diameter_step_connect_to_step_b" value="${4.17475704763*ratio_stl}" />
 </robot>

Commit message: adds step_c

File: xpider_ws/src/xpider_descriptions/models/xpider.xacro (robot description, xacro)
@@ -8,4 +8,5 @@
 <xacro:include filename="$(find xpider_descriptions)/models/step_connect.xacro"/>
 <xacro:include filename="$(find xpider_descriptions)/models/step_b.xacro"/>
+<xacro:include filename="$(find xpider_descriptions)/models/step_c.xacro"/>
 <xacro:include filename="$(find xpider_descriptions)/models/xpider.gazebo" />
 <!--<xacro:include filename="$(find xpider_descriptions)/models/leg_shield.xacro"/>-->
@@ -102,5 +103,5 @@
 	</joint>
   <xacro:step_b num="1"/>
-    <joint name="step_connect_2_to_step_b_2" type="fixed">
+  <joint name="step_connect_2_to_step_b_2" type="fixed">
 		<parent link="step_connect_2" />
 		<child link="step_b_2" />
@@ -108,5 +109,5 @@
 	</joint>
   <xacro:step_b num="2"/>
-    <joint name="step_connect_3_to_step_b_3" type="fixed">
+  <joint name="step_connect_3_to_step_b_3" type="fixed">
 		<parent link="step_connect_3" />
 		<child link="step_b_3" />
@@ -114,3 +115,21 @@
 	</joint>
   <xacro:step_b num="3"/>
+  <joint name="base_link_to_step_c_1" type="fixed">
+		<parent link="base_link" />
+		<child link="step_c_1" />
+    <origin xyz="${diameter_step_c*cos_m_pi_6} ${diameter_step_c*sin_m_pi_6} ${height_base_link_to_step_c}" rpy="0 0 0"/>
+	</joint>
+  <xacro:step_c num="1"/>
+  <joint name="base_link_to_step_c_2" type="fixed">
+		<parent link="base_link" />
+		<child link="step_c_2" />
+    <origin xyz="${diameter_step_c*cos_m_pi} ${diameter_step_c*sin_m_pi} ${height_base_link_to_step_c}" rpy="0 0 ${m_2_pi_3}"/>
+	</joint>
+  <xacro:step_c num="2"/>
+  <joint name="base_link_to_step_c_3" type="fixed">
+		<parent link="base_link" />
+		<child link="step_c_3" />
+    <origin xyz="${diameter_step_c*cos_m_5_pi_3} ${diameter_step_c*sin_m_5_pi_3} ${height_base_link_to_step_c}" rpy="0 0 ${2*m_2_pi_3}"/>
+	</joint>
+  <xacro:step_c num="3"/>
 </robot>

File: xpider_ws/src/xpider_resources/urdf/common_constants.xacro (robot description, xacro)
@@ -17,4 +17,8 @@
   <xacro:property name="cos_m_pi" value="-1" />
   <xacro:property name="sin_m_pi" value="0" />
+  <xacro:property name="cos_m_pi_2" value="0" />
+  <xacro:property name="sin_m_pi_2" value="1" />
+  <xacro:property name="cos_m_pi_6" value="0.5" />
+  <xacro:property name="sin_m_pi_6" value="0.86602540378" />
   <xacro:property name="cos_m_pi_3" value="0.5" />
   <xacro:property name="sin_m_pi_3" value="0.86602540378" />
@@ -25,4 +29,6 @@
   <xacro:property name="cos_m_5_pi_3" value="0.5" />
   <xacro:property name="sin_m_5_pi_3" value="-0.86602540378" />
+  <xacro:property name="cos_m_5_pi_6" value="-0.86602540378" />
+  <xacro:property name="sin_m_5_pi_6" value="0.5" />
   <xacro:property name="ratio_stl" value="0.01006046568"/>
   <xacro:property name="height_base" value="${48.705498889*ratio_stl}"/>
@@ -36,3 +42,5 @@
   <xacro:property name="height_step_connect_to_step_b" value="${3.99583888844*ratio_stl}" />
   <xacro:property name="diameter_step_connect_to_step_b" value="${4.17475704763*ratio_stl}" />
+  <xacro:property name="height_base_link_to_step_c" value="${base_link_to_step_height-0.99398977324*ratio_stl}"/>
+  <xacro:property name="diameter_step_c" value="${26*ratio_stl}" />
 </robot>

Commit message: adds legs 4 5 6

File: xpider_ws/src/xpider_descriptions/models/xpider.xacro (robot description, xacro)
@@ -133,3 +133,21 @@
 	</joint>
   <xacro:step_c num="3"/>
+  <joint name="base_link_to_leg_4" type="fixed">
+		<parent link="base_link" />
+		<child link="leg_4" />
+    <origin xyz="${diameter_step*cos_m_pi_3} ${diameter_step*sin_m_pi_3} ${base_link_to_step_height + height_leg}" rpy="0 0 ${m_pi_3}"/>
+	</joint>
+  <xacro:leg num="4"/>
+  <joint name="base_link_to_leg_5" type="fixed">
+		<parent link="base_link" />
+		<child link="leg_5" />
+    <origin xyz="${diameter_step*cos_m_pi} ${diameter_step*sin_m_pi} ${base_link_to_step_height + height_step/2}" rpy="0 0 ${m_pi}"/>
+	</joint>
+  <xacro:leg num="5"/>
+  <joint name="base_link_to_leg_6" type="fixed">
+		<parent link="base_link" />
+		<child link="leg_6" />
+    <origin xyz="${diameter_step*cos_m_5_pi_3} ${diameter_step*sin_m_5_pi_3} ${base_link_to_step_height + height_step/2}" rpy="0 0 ${-m_pi_3}"/>
+	</joint>
+  <xacro:leg num="6"/>
 </robot>

File: xpider_ws/src/xpider_resources/urdf/common_constants.xacro (robot description, xacro)
@@ -15,4 +15,5 @@
   <!-- Pi divided by six -->
   <xacro:property name="m_pi_6" value="0.52359877559" />
+  <xacro:property name="m_5_pi_3" value="${m_2_pi_3}" />
   <xacro:property name="cos_m_pi" value="-1" />
   <xacro:property name="sin_m_pi" value="0" />
