Commit message: updates base height, step_b orientation

File: xpider_ws/src/xpider_descriptions/models/step_b.xacro (robot description, xacro)
@@ -6,5 +6,5 @@
     <link name="step_b_${num}">
     <visual>
-      <origin xyz="0 0 0" rpy="-${m_pi_2} 0 ${m_pi}"/>
+      <origin xyz="0 0 0" rpy="${m_pi_3/10 - m_pi_2} 0 ${m_pi}"/>
       <geometry>
         <mesh filename="package://xpider_descriptions/meshes/step_b.stl" scale="${ratio_stl} ${ratio_stl} ${ratio_stl}"/>
@@ -13,5 +13,5 @@
       </visual>
       <collision>
-        <origin xyz="0 0 0" rpy="-${m_pi_2} 0 ${m_pi}"/>
+        <origin xyz="0 0 0" rpy="${m_pi_3/10 - m_pi_2} 0 ${m_pi}"/>
         <geometry>
           <mesh filename="package://xpider_descriptions/meshes/step_b.stl" scale="${ratio_stl} ${ratio_stl} ${ratio_stl}"/>

File: xpider_ws/src/xpider_descriptions/models/xpider.xacro (robot description, xacro)
@@ -136,5 +136,5 @@
 		<parent link="base_link" />
 		<child link="leg_4" />
-    <origin xyz="${diameter_step*cos_m_pi_3} ${diameter_step*sin_m_pi_3} ${base_link_to_step_height + height_leg}" rpy="0 0 ${m_pi_3}"/>
+    <origin xyz="${diameter_step*cos_m_pi_3} ${diameter_step*sin_m_pi_3} ${height_base_link_to_step_c}" rpy="0 0 ${m_pi_3}"/>
 	</joint>
   <xacro:leg num="4"/>
@@ -142,5 +142,5 @@
 		<parent link="base_link" />
 		<child link="leg_5" />
-    <origin xyz="${diameter_step*cos_m_pi} ${diameter_step*sin_m_pi} ${base_link_to_step_height + height_step/2}" rpy="0 0 ${m_pi}"/>
+    <origin xyz="${diameter_step*cos_m_pi} ${diameter_step*sin_m_pi} ${height_base_link_to_step_c}" rpy="0 0 ${m_pi}"/>
 	</joint>
   <xacro:leg num="5"/>
@@ -148,5 +148,5 @@
 		<parent link="base_link" />
 		<child link="leg_6" />
-    <origin xyz="${diameter_step*cos_m_5_pi_3} ${diameter_step*sin_m_5_pi_3} ${base_link_to_step_height + height_step/2}" rpy="0 0 ${-m_pi_3}"/>
+    <origin xyz="${diameter_step*cos_m_5_pi_3} ${diameter_step*sin_m_5_pi_3} ${height_base_link_to_step_c}" rpy="0 0 ${-m_pi_3}"/>
 	</joint>
   <xacro:leg num="6"/>

File: xpider_ws/src/xpider_resources/urdf/common_constants.xacro (robot description, xacro)
@@ -33,9 +33,9 @@
   <xacro:property name="sin_m_5_pi_6" value="0.5" />
   <xacro:property name="ratio_stl" value="0.01006046568"/>
-  <xacro:property name="height_base" value="${48.705498889*ratio_stl}"/>
-  <xacro:property name="height_step" value="0.04"/>
-  <xacro:property name="height_leg" value="${height_step/2 + 0.007}"/>
-  <xacro:property name="base_link_to_step_height" value="${height_base-0.28}"/>
-  <xacro:property name="base_link_to_step_up" value="${height_base - 0.05}"/>
+  <xacro:property name="height_base" value="${52*ratio_stl}"/>
+  <xacro:property name="height_step" value="${3.97595909298*ratio_stl}"/>
+  <xacro:property name="height_leg" value="${height_step/2 + 0*0.69579284127*ratio_stl}"/>
+  <xacro:property name="base_link_to_step_height" value="${height_base-27.8317136509*ratio_stl}"/>
+  <xacro:property name="base_link_to_step_up" value="${height_base - 4.96994886622*ratio_stl}"/>
   <xacro:property name="diameter_step" value="${53.7748467325*ratio_stl}" />
   <xacro:property name="diameter_step_up" value="${26*ratio_stl}" />
@@ -43,5 +43,5 @@
   <xacro:property name="height_step_connect_to_step_b" value="${3.99583888844*ratio_stl}" />
   <xacro:property name="diameter_step_connect_to_step_b" value="${4.17475704763*ratio_stl}" />
-  <xacro:property name="height_base_link_to_step_c" value="${base_link_to_step_height-0.99398977324*ratio_stl}"/>
+  <xacro:property name="height_base_link_to_step_c" value="${base_link_to_step_height-1.6*ratio_stl}"/>
   <xacro:property name="diameter_step_c" value="${26*ratio_stl}" />
 </robot>

Commit message: updates leg and step_b orientation to match holes

File: xpider_ws/src/xpider_descriptions/models/step_b.xacro (robot description, xacro)
@@ -6,5 +6,5 @@
     <link name="step_b_${num}">
     <visual>
-      <origin xyz="0 0 0" rpy="${m_pi_3/10 - m_pi_2} 0 ${m_pi}"/>
+      <origin xyz="0 0 0" rpy="${m_pi_3/11 - m_pi_2} 0 ${m_pi}"/>
       <geometry>
         <mesh filename="package://xpider_descriptions/meshes/step_b.stl" scale="${ratio_stl} ${ratio_stl} ${ratio_stl}"/>
@@ -13,5 +13,5 @@
       </visual>
       <collision>
-        <origin xyz="0 0 0" rpy="${m_pi_3/10 - m_pi_2} 0 ${m_pi}"/>
+        <origin xyz="0 0 0" rpy="${m_pi_3/11 - m_pi_2} 0 ${m_pi}"/>
         <geometry>
           <mesh filename="package://xpider_descriptions/meshes/step_b.stl" scale="${ratio_stl} ${ratio_stl} ${ratio_stl}"/>

File: xpider_ws/src/xpider_descriptions/models/xpider.xacro (robot description, xacro)
@@ -142,5 +142,5 @@
 		<parent link="base_link" />
 		<child link="leg_5" />
-    <origin xyz="${diameter_step*cos_m_pi} ${diameter_step*sin_m_pi} ${height_base_link_to_step_c}" rpy="0 0 ${m_pi}"/>
+    <origin xyz="${diameter_step*cos_m_pi} ${diameter_step*sin_m_pi} ${height_base_link_to_step_c}" rpy="0 0.07 ${m_pi}"/>
 	</joint>
   <xacro:leg num="5"/>
