Commit message: Each leg can be moved with joint state publisher.

File: xpider_ws/src/xpider_descriptions/models/step_c.xacro (robot description, xacro)
@@ -6,5 +6,5 @@
     <link name="step_c_${num}">
     <visual>
-      <origin xyz="0 0 0" rpy="-${m_pi_2} 0 ${m_pi_3}"/>
+      <origin xyz="0 0 0" rpy="-${m_pi_2} 0 ${m_pi_3 + m_pi_6}"/>
       <geometry>
         <mesh filename="package://xpider_descriptions/meshes/step_c.stl" scale="${ratio_stl} ${ratio_stl} ${ratio_stl}"/>
@@ -13,5 +13,5 @@
       </visual>
       <collision>
-        <origin xyz="0 0 0" rpy="-${m_pi_2} 0 ${m_pi_3}"/>
+        <origin xyz="0 0 0" rpy="-${m_pi_2} 0 ${m_pi_3 + m_pi_6}"/>
         <geometry>
           <mesh filename="package://xpider_descriptions/meshes/step_c.stl" scale="${ratio_stl} ${ratio_stl} ${ratio_stl}"/>

File: xpider_ws/src/xpider_descriptions/models/step_up.xacro (robot description, xacro)
@@ -6,5 +6,5 @@
     <link name="step_up_${num}">
     <visual>
-      <origin xyz="0 0 0" rpy="${m_pi_2-0.2} 0 ${m_pi_3+m_pi_6}"/>
+      <origin xyz="0 0 0" rpy="${m_pi_2} 0 ${m_pi_3+m_pi_6}"/>
       <geometry>
         <mesh filename="package://xpider_descriptions/meshes/step_up.stl" scale="${ratio_stl} ${ratio_stl} ${ratio_stl}"/>
@@ -13,5 +13,5 @@
       </visual>
       <collision>
-        <origin xyz="0 0 0" rpy="${m_pi_2-0.2} 0 ${m_pi_3+m_pi_6}"/>
+        <origin xyz="0 0 0" rpy="${m_pi_2} 0 ${m_pi_3+m_pi_6}"/>
         <geometry>
           <mesh filename="package://xpider_descriptions/meshes/step_up.stl" scale="${ratio_stl} ${ratio_stl} ${ratio_stl}"/>

File: xpider_ws/src/xpider_descriptions/models/xpider.xacro (robot description, xacro)
@@ -12,142 +12,9 @@
 <!--<xacro:include filename="$(find xpider_descriptions)/models/leg_shield.xacro"/>-->
   <link name="world"/>
-  <joint name="fixed" type="fixed">
-    <parent link="world"/>
-    <child link="base_link"/>
-  </joint>
-  <xacro:include filename="$(find xpider_descriptions)/models/base_link.xacro"/>
-  <joint name="base_joint" type="fixed">
-		<parent link="base_link" />
-		<child link="shield_top" />
-		<origin xyz="0 0 ${height_base}" rpy="0 0 ${m_pi_3}" /> <!-- TOCHECK-->
-	</joint>
-  <xacro:include filename="$(find xpider_descriptions)/models/shield_top.xacro"/>
-  <joint name="base_joint2" type="fixed">
-		<parent link="base_link" />
-		<child link="shield_bottom" />
-		<origin xyz="0 0 ${height_base}" rpy="0 0 ${m_pi_3 + m_pi_6}" />
-	</joint>
-  <xacro:include filename="$(find xpider_descriptions)/models/shield_bottom.xacro"/>
-  <joint name="base_joint3" type="fixed">
-		<parent link="base_link" />
-		<child link="step" />
-		<origin xyz="0 0 ${base_link_to_step_height + height_step/2}" rpy="0 0 ${m_pi_2 + m_pi_6}" />
-	</joint>
-   <xacro:include filename="$(find xpider_descriptions)/models/step.xacro"/>
-  <joint name="base_joint4" type="fixed">
-		<parent link="base_link" />
-		<child link="step_base" />
-		<origin xyz="0 0 ${height_base}" rpy="0 0 ${m_pi_3 + m_pi_6}" />
-	</joint>
-  <xacro:include filename="$(find xpider_descriptions)/models/step_base.xacro"/>
+  <!-- Big fixed components-->
+  <xacro:include filename="$(find xpider_descriptions)/models/set_base.xacro" />
   <!--  First set of Legs -->
-  <joint name="base_link_to_leg_1" type="fixed">
-		<parent link="base_link" />
-		<child link="leg_1" />
-    <origin xyz="${diameter_step} 0 ${base_link_to_step_height + height_leg}" rpy="0 0 0"/>
-	</joint>
-  <xacro:leg num="1"/>
-  <joint name="base_link_to_leg_2" type="fixed">
-		<parent link="base_link" />
-		<child link="leg_2" />
-    <origin xyz="${diameter_step*cos_m_2_pi_3} ${diameter_step*sin_m_2_pi_3} ${base_link_to_step_height + height_step/2}" rpy="0 0 ${m_2_pi_3}"/>
-	</joint>
-  <xacro:leg num="2"/>
-  <joint name="base_link_to_leg_3" type="fixed">
-		<parent link="base_link" />
-		<child link="leg_3" />
-    <origin xyz="${diameter_step*cos_m_4_pi_3} ${diameter_step*sin_m_4_pi_3} ${base_link_to_step_height + height_step/2}" rpy="0 0 ${2*m_2_pi_3}"/>
-	</joint>
-  <xacro:leg num="3"/>
-  <joint name="base_link_to_step_up_1" type="fixed">
-		<parent link="base_link" />
-		<child link="step_up_1" />
-    <origin xyz="${diameter_step_up} 0 ${base_link_to_step_up}" rpy="0 ${m_pi_6} 0"/>
-	</joint>
-  <xacro:step_up num="1"/>
-  <joint name="base_link_to_step_up_2" type="fixed">
-		<parent link="base_link" />
-		<child link="step_up_2" />
-    <origin xyz="${diameter_step_up*cos_m_2_pi_3} ${diameter_step_up*sin_m_2_pi_3} ${base_link_to_step_up}" rpy="0 ${m_pi_6} ${m_2_pi_3}"/>
-	</joint>
-  <xacro:step_up num="2"/>
-  <joint name="base_link_to_step_up_3" type="fixed">
-		<parent link="base_link" />
-		<child link="step_up_3" />
-    <origin xyz="${diameter_step_up*cos_m_4_pi_3} ${diameter_step_up*sin_m_4_pi_3} ${base_link_to_step_up}" rpy="0 ${m_pi_6} ${2*m_2_pi_3}"/>
-	</joint>
-  <xacro:step_up num="3"/>
- <!-- Second set of legs -->
-  <joint name="base_link_to_step_connect_1" type="fixed">
-		<parent link="base_link" />
-		<child link="step_connect_1" />
-    <origin xyz="${diameter_step_connect*cos_m_pi_3} ${diameter_step_connect*sin_m_pi_3} ${base_link_to_step_height + 0.0624}" rpy="0 0 ${-m_pi_6}"/>
-	</joint>
-  <xacro:step_connect num="1"/>
-  <joint name="base_link_to_step_connect_2" type="fixed">
-		<parent link="base_link" />
-		<child link="step_connect_2" />
-    <origin xyz="${diameter_step_connect*cos_m_pi} ${diameter_step_connect*sin_m_pi} ${base_link_to_step_height + 0.0624}" rpy="0 0 ${-m_pi_6 + m_2_pi_3}"/>
-	</joint>
-  <xacro:step_connect num="2"/>
-  <joint name="base_link_to_step_connect_3" type="fixed">
-		<parent link="base_link" />
-		<child link="step_connect_3" />
-    <origin xyz="${diameter_step_connect*cos_m_5_pi_3} ${diameter_step_connect*sin_m_5_pi_3} ${base_link_to_step_height + 0.0624}" rpy="0 0 ${-m_pi_6 + 2*m_2_pi_3}"/>
-	</joint>
-  <xacro:step_connect num="3"/>
-  <joint name="step_connect_1_to_step_b_1" type="fixed">
-		<parent link="step_connect_1" />
-		<child link="step_b_1" />
-    <origin xyz="${0} ${0.042} ${0.0402}" rpy="0 0 ${0}"/>
-	</joint>
-  <xacro:step_b num="1"/>
-  <joint name="step_connect_2_to_step_b_2" type="fixed">
-		<parent link="step_connect_2" />
-		<child link="step_b_2" />
-    <origin xyz="${0} ${diameter_step_connect_to_step_b} ${height_step_connect_to_step_b}" rpy="0 0 0"/>
-	</joint>
-  <xacro:step_b num="2"/>
-  <joint name="step_connect_3_to_step_b_3" type="fixed">
-		<parent link="step_connect_3" />
-		<child link="step_b_3" />
-    <origin xyz="${0} ${diameter_step_connect_to_step_b} ${height_step_connect_to_step_b}" rpy="0 0 0"/>
-	</joint>
-  <xacro:step_b num="3"/>
-  <joint name="base_link_to_step_c_1" type="fixed">
-		<parent link="base_link" />
-		<child link="step_c_1" />
-    <origin xyz="${diameter_step_c*cos_m_pi_6} ${diameter_step_c*sin_m_pi_6} ${height_base_link_to_step_c}" rpy="0 0 0"/>
-	</joint>
-  <xacro:step_c num="1"/>
-  <joint name="base_link_to_step_c_2" type="fixed">
-		<parent link="base_link" />
-		<child link="step_c_2" />
-    <origin xyz="${diameter_step_c*cos_m_pi} ${diameter_step_c*sin_m_pi} ${height_base_link_to_step_c}" rpy="0 0 ${m_2_pi_3}"/>
-	</joint>
-  <xacro:step_c num="2"/>
-  <joint name="base_link_to_step_c_3" type="fixed">
-		<parent link="base_link" />
-		<child link="step_c_3" />
-    <origin xyz="${diameter_step_c*cos_m_5_pi_3} ${diameter_step_c*sin_m_5_pi_3} ${height_base_link_to_step_c}" rpy="0 0 ${2*m_2_pi_3}"/>
-	</joint>
-  <xacro:step_c num="3"/>
-  <joint name="base_link_to_leg_4" type="fixed">
-		<parent link="base_link" />
-		<child link="leg_4" />
-    <origin xyz="${diameter_step*cos_m_pi_3} ${diameter_step*sin_m_pi_3} ${height_base_link_to_step_c}" rpy="0 0 ${m_pi_3}"/>
-	</joint>
-  <xacro:leg num="4"/>
-  <joint name="base_link_to_leg_5" type="fixed">
-		<parent link="base_link" />
-		<child link="leg_5" />
-    <origin xyz="${diameter_step*cos_m_pi} ${diameter_step*sin_m_pi} ${height_base_link_to_step_c}" rpy="0 0.07 ${m_pi}"/>
-	</joint>
-  <xacro:leg num="5"/>
-  <joint name="base_link_to_leg_6" type="fixed">
-		<parent link="base_link" />
-		<child link="leg_6" />
-    <origin xyz="${diameter_step*cos_m_5_pi_3} ${diameter_step*sin_m_5_pi_3} ${height_base_link_to_step_c}" rpy="0 0 ${-m_pi_3}"/>
-	</joint>
-  <xacro:leg num="6"/>
+  <xacro:include filename="$(find xpider_descriptions)/models/set_legs_1.xacro" />
+  <!-- Second set of legs -->
+  <xacro:include filename="$(find xpider_descriptions)/models/set_legs_2.xacro" />
 </robot>

File: xpider_ws/src/xpider_resources/urdf/common_constants.xacro (robot description, xacro)
@@ -38,5 +38,6 @@
   <xacro:property name="base_link_to_step_height" value="${height_base-27.8317136509*ratio_stl}"/>
   <xacro:property name="base_link_to_step_up" value="${height_base - 4.96994886622*ratio_stl}"/>
-  <xacro:property name="diameter_step" value="${53.7748467325*ratio_stl}" />
+  <xacro:property name="diameter_step" value="${47*ratio_stl}" />
+  <xacro:property name="diameter_step_up_to_leg" value="${31.5*ratio_stl}" />
   <xacro:property name="diameter_step_up" value="${26*ratio_stl}" />
   <xacro:property name="diameter_step_connect" value="${5.5*ratio_stl}" />
