Commit message: adds leg shields

File: xpider_ws/src/xpider_descriptions/models/leg_shield.xacro (robot description, xacro)
@@ -6,5 +6,5 @@
       <link name="leg_shield_${num}">
       <visual>
-        <origin xyz="-${diameter_step-0.052} -0.198 0" rpy="0 0 -0.2"/>
+        <origin xyz="0 0 0" rpy="0 0 0"/>
         <geometry>
           <mesh filename="package://xpider_descriptions/meshes/leg_shield.stl" scale="${ratio_stl} ${ratio_stl} ${ratio_stl}"/>
@@ -13,5 +13,5 @@
         </visual>
         <collision>
-          <origin xyz="-${diameter_step-0.052} -0.198 0" rpy="0 0 -0.2"/>
+          <origin xyz="0 0 0" rpy="0 0 0"/>
           <geometry>
             <mesh filename="package://xpider_descriptions/meshes/leg_shield.stl" scale="${ratio_stl} ${ratio_stl} ${ratio_stl}"/>

File: xpider_ws/src/xpider_descriptions/models/xpider.xacro (robot description, xacro)
@@ -17,3 +17,5 @@
   <!-- Second set of legs -->
   <xacro:include filename="$(find xpider_descriptions)/models/set_legs_2.xacro" />
+  <!-- Leg shields -->
+  <xacro:include filename="$(find xpider_descriptions)/models/set_legs_shield.xacro" />
 </robot>

File: xpider_ws/src/xpider_resources/urdf/common_constants.xacro (robot description, xacro)
@@ -54,3 +54,6 @@
   <xacro:property name="step_to_step_connect_height" value="${6.20249618505*ratio_stl}"/>
   <xacro:property name="diameter_step_c" value="${26*ratio_stl}" />
+  <xacro:property name="x_leg_to_leg_shield_set_1" value="${2.48497443311*ratio_stl}" />
+  <xacro:property name="x_leg_to_leg_shield_set_2" value="${1.49098465987*ratio_stl}" />
+  <xacro:property name="z_leg_to_leg_shield" value="${5.96393863947*ratio_stl}" />
 </robot>
