Commit message: legs 1 2 3 are children of step

File: xpider_ws/src/xpider_descriptions/models/set_base.xacro (robot description, xacro)
@@ -19,11 +19,13 @@
 	</joint>
   <xacro:include filename="$(find xpider_descriptions)/models/shield_bottom.xacro"/>
-  <joint name="base_joint3" type="fixed">
+  <joint name="base_step" type="prismatic">
 		<parent link="base_link" />
 		<child link="step" />
 		<origin xyz="0 0 ${base_link_to_step_height + height_step/2}" rpy="0 0 ${m_pi_2 + m_pi_6}" />
+    <limit effort="1000.0" lower="0" upper="0.03" velocity="0.5"/>
+    <axis xyz="0 0 1"/>
 	</joint>
-   <xacro:include filename="$(find xpider_descriptions)/models/step.xacro"/>
-  <joint name="base_joint4" type="fixed">
+  <xacro:include filename="$(find xpider_descriptions)/models/step.xacro"/>
+  <joint name="base_step_base" type="fixed">
 		<parent link="base_link" />
 		<child link="step_base" />

File: xpider_ws/src/xpider_descriptions/models/set_legs_1.xacro (robot description, xacro)
@@ -1,10 +1,13 @@
 <?xml version="1.0" ?>
 <robot name="xpider_set_legs_1" xmlns:xacro="http://ros.org/wiki/xacro">
+<xacro:include filename="$(find xpider_descriptions)/models/leg.xacro"/>
+<xacro:include filename="$(find xpider_descriptions)/models/leg2.xacro"/>
   <joint name="base_link_to_step_up_1" type="revolute">
 		<parent link="base_link" />
 		<child link="step_up_1" />
-    <origin xyz="${diameter_step_up} 0 ${base_link_to_step_up}" rpy="0 ${m_pi_6/2} 0"/>
-    <limit effort="1000.0" lower="-0.1" upper="0.1" velocity="0.5"/>
-    <axis xyz="0 1 0"/>
+    <origin xyz="${diameter_step_up} 0 ${base_link_to_step_up}" rpy="${m_pi_2 + 0.38} ${0} ${m_pi_3+m_pi_6}"/>
+    <limit effort="1000.0" lower="0" upper="1" velocity="0.5"/>
+    <axis xyz="1 0 0"/>
+    <mimic joint="base_step" multiplier="-5" offset="0" />
 	</joint>
   <xacro:step_up num="1"/>
@@ -12,7 +15,8 @@
 		<parent link="base_link" />
 		<child link="step_up_2" />
-    <origin xyz="${diameter_step_up*cos_m_2_pi_3} ${diameter_step_up*sin_m_2_pi_3} ${base_link_to_step_up}" rpy="0 ${m_pi_6/2} ${m_2_pi_3}"/>
-    <limit effort="1000.0" lower="-0.1" upper="0.1" velocity="0.5"/>
-    <axis xyz="0 1 0"/>
+    <origin xyz="${diameter_step_up*cos_m_2_pi_3} ${diameter_step_up*sin_m_2_pi_3} ${base_link_to_step_up}" rpy="${m_pi_2 + 0.38} ${0} ${m_2_pi_3 + m_pi_3+m_pi_6}"/>
+    <limit effort="1000.0" lower="0" upper="1" velocity="0.5"/>
+    <axis xyz="1 0 0"/>
+    <mimic joint="base_step" multiplier="-5" offset="0" />
 	</joint>
   <xacro:step_up num="2"/>
@@ -20,26 +24,36 @@
 		<parent link="base_link" />
 		<child link="step_up_3" />
-    <origin xyz="${diameter_step_up*cos_m_4_pi_3} ${diameter_step_up*sin_m_4_pi_3} ${base_link_to_step_up}" rpy="0 ${m_pi_6/2} ${2*m_2_pi_3}"/>
-    <limit effort="1000.0" lower="-0.1" upper="0.1" velocity="0.5"/>
-    <axis xyz="0 1 0"/>
+    <origin xyz="${diameter_step_up*cos_m_4_pi_3} ${diameter_step_up*sin_m_4_pi_3} ${base_link_to_step_up}" rpy="${m_pi_2 + 0.38} ${0} ${2*m_2_pi_3 + m_pi_3+m_pi_6}"/>
+    <limit effort="1000.0" lower="0" upper="1" velocity="0.5"/>
+    <axis xyz="1 0 0"/>
+    <mimic joint="base_step" multiplier="-5" offset="0" />
 	</joint>
   <xacro:step_up num="3"/>
-  <joint name="step_up_1_to_leg_1" type="fixed">
-		<parent link="step_up_1" />
+  <joint name="step_to_leg_1" type="revolute">
+		<parent link="step" />
 		<child link="leg_1" />
-    <origin xyz="${diameter_step_up_to_leg} ${0} ${0.007}" rpy="0 ${-m_pi/16} 0"/>
+    <origin xyz="${diameter_step_to_leg_123*cos_m_4_pi_3} ${diameter_step_to_leg_123*sin_m_4_pi_3} ${0}" rpy="0 0.18 ${-m_2_pi_3}"/>
+    <limit effort="1000.0" lower="0" upper="1" velocity="0.5"/>
+    <axis xyz="0 1 0"/>
+    <mimic joint="base_step" multiplier="2" offset="0" />
 	</joint>
-  <xacro:leg num="1"/>
-  <joint name="step_up_2_to_leg_2" type="fixed">
-		<parent link="step_up_2" />
+  <xacro:leg2 num="1"/>
+  <joint name="step_to_leg_2" type="revolute">
+		<parent link="step" />
 		<child link="leg_2" />
-    <origin xyz="${diameter_step_up_to_leg} ${0} ${0.007}" rpy="0 ${-m_pi/16} 0"/>
+    <origin xyz="${diameter_step_to_leg_123} ${diameter_step_to_leg_123*0} ${0}" rpy="0 0.18 ${0}"/>
+    <limit effort="1000.0" lower="0" upper="1" velocity="0.5"/>
+    <axis xyz="0 1 0"/>
+    <mimic joint="base_step" multiplier="2" offset="0" />
 	</joint>
-  <xacro:leg num="2"/>
-  <joint name="step_up_3_to_leg_3" type="fixed">
-		<parent link="step_up_3" />
+  <xacro:leg2 num="2"/>
+  <joint name="step_to_leg_3" type="revolute">
+		<parent link="step" />
 		<child link="leg_3" />
-    <origin xyz="${diameter_step_up_to_leg} ${0} ${0.007}" rpy="0 ${-m_pi/16} 0"/>
+    <origin xyz="${diameter_step_to_leg_123*cos_m_2_pi_3} ${diameter_step_to_leg_123*sin_m_2_pi_3} ${0}" rpy="0 0.18 ${-2*m_2_pi_3}"/>
+    <limit effort="1000.0" lower="0" upper="1" velocity="0.5"/>
+    <axis xyz="0 1 0"/>
+    <mimic joint="base_step" multiplier="2" offset="0" />
 	</joint>
-  <xacro:leg num="3"/>
+  <xacro:leg2 num="3"/>
 </robot>

File: xpider_ws/src/xpider_descriptions/models/set_legs_2.xacro (robot description, xacro)
@@ -1,4 +1,6 @@
 <?xml version="1.0" ?>
 <robot name="xpider_set_legs_2" xmlns:xacro="http://ros.org/wiki/xacro">
+<xacro:include filename="$(find xpider_descriptions)/models/leg.xacro"/>
+<xacro:include filename="$(find xpider_descriptions)/models/leg2.xacro"/>
   <joint name="base_link_to_step_connect_1" type="fixed">
  		<parent link="base_link" />

File: xpider_ws/src/xpider_descriptions/models/step_up.xacro (robot description, xacro)
@@ -6,5 +6,5 @@
     <link name="step_up_${num}">
     <visual>
-      <origin xyz="0 0 0" rpy="${m_pi_2} 0 ${m_pi_3+m_pi_6}"/>
+      <origin xyz="0 0 0" rpy="0 0 0"/>
       <geometry>
         <mesh filename="package://xpider_descriptions/meshes/step_up.stl" scale="${ratio_stl} ${ratio_stl} ${ratio_stl}"/>
@@ -13,5 +13,5 @@
       </visual>
       <collision>
-        <origin xyz="0 0 0" rpy="${m_pi_2} 0 ${m_pi_3+m_pi_6}"/>
+        <origin xyz="0 0 0" rpy="0 0 0"/>
         <geometry>
           <mesh filename="package://xpider_descriptions/meshes/step_up.stl" scale="${ratio_stl} ${ratio_stl} ${ratio_stl}"/>

File: xpider_ws/src/xpider_descriptions/models/xpider.xacro (robot description, xacro)
@@ -4,5 +4,4 @@
 <xacro:include filename="$(find xpider_resources)/urdf/common_constants.xacro"/>
 <xacro:include filename="$(find xpider_descriptions)/models/step_bridge.xacro"/>
-<xacro:include filename="$(find xpider_descriptions)/models/leg.xacro"/>
 <xacro:include filename="$(find xpider_descriptions)/models/step_up.xacro"/>
 <xacro:include filename="$(find xpider_descriptions)/models/step_connect.xacro"/>

File: xpider_ws/src/xpider_resources/urdf/common_constants.xacro (robot description, xacro)
@@ -32,4 +32,6 @@
   <xacro:property name="cos_m_5_pi_6" value="-0.86602540378" />
   <xacro:property name="sin_m_5_pi_6" value="0.5" />
+  <xacro:property name="cos_m_11_pi_6" value="0.86602540378" />
+  <xacro:property name="sin_m_11_pi_6" value="-0.5" />
   <xacro:property name="ratio_stl" value="0.01006046568"/>
   <xacro:property name="height_base" value="${52*ratio_stl}"/>
@@ -39,4 +41,5 @@
   <xacro:property name="base_link_to_step_up" value="${height_base - 4.96994886622*ratio_stl}"/>
   <xacro:property name="diameter_step" value="${47*ratio_stl}" />
+  <xacro:property name="diameter_step_to_leg_123" value="${54*ratio_stl}" />
   <xacro:property name="diameter_step_up_to_leg" value="${31.5*ratio_stl}" />
   <xacro:property name="diameter_step_up" value="${26*ratio_stl}" />

Commit message: xpider_descriptions.cpp: sets joints at start

File: xpider_ws/src/xpider_descriptions/models/set_base.xacro (robot description, xacro)
@@ -6,5 +6,5 @@
   </joint>
   <xacro:include filename="$(find xpider_descriptions)/models/base_link.xacro"/>
-  <joint name="base_joint" type="continuous">
+  <joint name="base_link_to_shield_top" type="continuous">
 		<parent link="base_link" />
 		<child link="shield_top" />
