Commit message: use parameter server to initialize position of each joint

File: xpider_descriptions/models/set_base.xacro (robot description, xacro)
@@ -19,13 +19,13 @@
 	</joint>
   <xacro:include filename="$(find xpider_descriptions)/models/shield_bottom.xacro"/>
-  <joint name="base_step" type="prismatic">
+  <joint name="base_link_to_step" type="prismatic">
 		<parent link="base_link" />
 		<child link="step" />
 		<origin xyz="0 0 ${base_link_to_step_height + height_step/2}" rpy="0 0 ${m_pi_2 + m_pi_6}" />
-    <limit effort="1000.0" lower="0" upper="0.03" velocity="0.5"/>
+    <limit effort="1000.0" lower="0" upper="0.06" velocity="0.5"/>
     <axis xyz="0 0 1"/>
 	</joint>
   <xacro:include filename="$(find xpider_descriptions)/models/step.xacro"/>
-  <joint name="base_step_base" type="fixed">
+  <joint name="base_link_to_step_base" type="fixed">
 		<parent link="base_link" />
 		<child link="step_base" />

File: xpider_descriptions/models/set_legs_1.xacro (robot description, xacro)
@@ -9,5 +9,5 @@
     <limit effort="1000.0" lower="0" upper="1" velocity="0.5"/>
     <axis xyz="1 0 0"/>
-    <mimic joint="base_step" multiplier="-5" offset="0" />
+    <mimic joint="base_link_to_step" multiplier="-5" offset="0" />
 	</joint>
   <xacro:step_up num="1"/>
@@ -18,5 +18,5 @@
     <limit effort="1000.0" lower="0" upper="1" velocity="0.5"/>
     <axis xyz="1 0 0"/>
-    <mimic joint="base_step" multiplier="-5" offset="0" />
+    <mimic joint="base_link_to_step" multiplier="-5" offset="0" />
 	</joint>
   <xacro:step_up num="2"/>
@@ -27,5 +27,5 @@
     <limit effort="1000.0" lower="0" upper="1" velocity="0.5"/>
     <axis xyz="1 0 0"/>
-    <mimic joint="base_step" multiplier="-5" offset="0" />
+    <mimic joint="base_link_to_step" multiplier="-5" offset="0" />
 	</joint>
   <xacro:step_up num="3"/>
@@ -36,5 +36,5 @@
     <limit effort="1000.0" lower="0" upper="1" velocity="0.5"/>
     <axis xyz="0 1 0"/>
-    <mimic joint="base_step" multiplier="2" offset="0" />
+    <mimic joint="base_link_to_step" multiplier="2" offset="0" />
 	</joint>
   <xacro:leg2 num="1"/>
@@ -45,5 +45,5 @@
     <limit effort="1000.0" lower="0" upper="1" velocity="0.5"/>
     <axis xyz="0 1 0"/>
-    <mimic joint="base_step" multiplier="2" offset="0" />
+    <mimic joint="base_link_to_step" multiplier="2" offset="0" />
 	</joint>
   <xacro:leg2 num="2"/>
@@ -54,5 +54,5 @@
     <limit effort="1000.0" lower="0" upper="1" velocity="0.5"/>
     <axis xyz="0 1 0"/>
-    <mimic joint="base_step" multiplier="2" offset="0" />
+    <mimic joint="base_link_to_step" multiplier="2" offset="0" />
 	</joint>
   <xacro:leg2 num="3"/>

File: xpider_descriptions/models/set_legs_2.xacro (robot description, xacro)
@@ -32,5 +32,5 @@
     <origin xyz="${0} ${diameter_step_connect_to_step_b} ${height_step_connect_to_step_b}" rpy="0 0 0"/>
     <axis xyz="1 0 0"/>
-    <limit effort="1000.0" lower="-0.1" upper="-0.04" velocity="0.5"/>
+    <limit effort="1000.0" lower="-0.1" upper="0.08" velocity="0.5"/>
  	</joint>
    <xacro:step_b num="1"/>
@@ -40,5 +40,5 @@
     <origin xyz="${0} ${diameter_step_connect_to_step_b} ${height_step_connect_to_step_b}" rpy="0 0 0"/>
     <axis xyz="1 0 0"/>
-    <limit effort="1000.0" lower="-0.1" upper="-0.04" velocity="0.5"/>
+    <limit effort="1000.0" lower="-0.1" upper="0.08" velocity="0.5"/>
  	</joint>
    <xacro:step_b num="2"/>
@@ -48,5 +48,5 @@
     <origin xyz="${0} ${diameter_step_connect_to_step_b} ${height_step_connect_to_step_b}" rpy="0 0 0"/>
     <axis xyz="1 0 0"/>
-    <limit effort="1000.0" lower="-0.1" upper="-0.04" velocity="0.5"/>
+    <limit effort="1000.0" lower="-0.1" upper="0.08" velocity="0.5"/>
  	</joint>
    <xacro:step_b num="3"/>
